Commit message: Fix collision and visual colors for Gazebo Fortress
- Move self_collide to model level (no reference attr): in SDF 1.9 it is a
  model attribute; per-link self_collide inside <gazebo reference> is ignored
  by Fortress, causing the arm to pass through the base plate
- Add Ogre2 RGBA grey material to base_plate_02_link (Gazebo/White invalid)
- Add Ogre2 RGBA black material for all 8 arm links via gz_black macro
  (Gazebo/DarkGrey from upstream gazebo.xacro is Ogre1 and ignored by Fortress)

Co-Authored-By: Claude Sonnet 4.6 <noreply@anthropic.com>

File: xacro/open_manipulator_x_effort_robot.urdf.xacro (robot description, xacro)
@@ -60,7 +60,12 @@
     </inertial>
   </link>
-  <!-- Propiedades de contacto Gazebo para la placa.
-       self_collide permite que el brazo colisione con la placa (intra-modelo).
-       Nota: material Gazebo/White eliminado — no existe en Ogre2 (Fortress). -->
+  <!-- Colision intra-modelo (brazo vs placa): self_collide es un atributo de
+       nivel de modelo en SDF 1.9 (Fortress). Debe ir en <gazebo> sin reference.
+       El <self_collide> dentro de <gazebo reference="..."> es ignorado en Fortress. -->
+  <gazebo>
+    <self_collide>true</self_collide>
+  </gazebo>
+  <!-- Propiedades de contacto y color (gris) para la placa base.
+       Material en formato RGBA Ogre2 — Gazebo/White no existe en Fortress. -->
   <gazebo reference="base_plate_02_link">
     <kp>1000000.0</kp>
@@ -68,6 +73,34 @@
     <mu1>0.6</mu1>
     <mu2>0.6</mu2>
-    <self_collide>true</self_collide>
+    <visual>
+      <material>
+        <ambient>0.5 0.5 0.5 1</ambient>
+        <diffuse>0.5 0.5 0.5 1</diffuse>
+        <specular>0.1 0.1 0.1 1</specular>
+      </material>
+    </visual>
   </gazebo>
+  <!-- Colores Ogre2 (Fortress) para los eslabones del brazo: negro.
+       Los <material>Gazebo/DarkGrey</material> del paquete externo son Ogre1
+       y son ignorados por Fortress. Estos bloques los reemplazan. -->
+  <xacro:macro name="gz_black" params="link">
+    <gazebo reference="${link}">
+      <visual>
+        <material>
+          <ambient>0.05 0.05 0.05 1</ambient>
+          <diffuse>0.1  0.1  0.1  1</diffuse>
+          <specular>0.1  0.1  0.1  1</specular>
+        </material>
+      </visual>
+    </gazebo>
+  </xacro:macro>
+  <xacro:gz_black link="$(arg prefix)link1"/>
+  <xacro:gz_black link="$(arg prefix)link2"/>
+  <xacro:gz_black link="$(arg prefix)link3"/>
+  <xacro:gz_black link="$(arg prefix)link4"/>
+  <xacro:gz_black link="$(arg prefix)link5"/>
+  <xacro:gz_black link="$(arg prefix)gripper_left_link"/>
+  <xacro:gz_black link="$(arg prefix)gripper_right_link"/>
+  <xacro:gz_black link="$(arg prefix)end_effector_link"/>
   <!-- Placa anclada directamente al mundo. Ambos joints van a world para que
        Gazebo no fusione base_plate_02_link con link1 al convertir URDF→SDF. -->

Commit message: xacro/sim: add load_x_offset to shift cylinder along end_effector X axis
Nuevo parametro load_x_offset [m] (default 0.0) que traslada el centro
del cilindro a lo largo del eje X del frame end_effector_link, modificando
el joint origin del load_joint. Permite simular cargas descentradas.

Archivos: xacro/open_manipulator_x_effort_robot.urdf.xacro
          config/sim_init_config.yaml
          launch/torque_sim.launch.py

Co-Authored-By: Claude Sonnet 4.6 <noreply@anthropic.com>

File: xacro/open_manipulator_x_effort_robot.urdf.xacro (robot description, xacro)
@@ -18,4 +18,10 @@
   <xacro:arg name="mass_inertia_scale" default="1.0" />
   <xacro:arg name="damping_scale"      default="1.0" />
+  <!-- Carga cilindrica en el efector final: configurables desde sim_init_config.yaml -->
+  <xacro:arg name="spawn_load"    default="false" />
+  <xacro:arg name="load_radius"   default="0.05"  />   <!-- radio         [m] -->
+  <xacro:arg name="load_height"   default="0.02"  />   <!-- altura        [m] -->
+  <xacro:arg name="load_mass"     default="0.1"   />   <!-- masa          [kg] -->
+  <xacro:arg name="load_x_offset" default="0.0"   />   <!-- offset en X   [m] -->
   <!-- Recursos graficos: colores Rviz y materiales Gazebo del paquete original -->
   <xacro:include filename="$(find open_manipulator_x_description)/gazebo/materials.xacro" />
@@ -137,3 +143,58 @@
     <child link="$(arg prefix)link1"/>
   </joint>
+  <!-- ── Carga cilindrica en el efector final ──────────────────────────────────
+       Cilindro solido cuyo eje coincide con el eje Y de end_effector_link.
+       Las caras circulares apuntan en +Y / -Y (rpy pi/2 0 0 alinea eje Z→Y).
+       Inercia de cilindro solido con eje a lo largo de Y:
+         Ixx = Izz = m*(3r^2 + h^2)/12
+         Iyy = m*r^2/2
+       Solo se instancia si spawn_load:=true; en caso contrario no existe en
+       el arbol cinematico y no afecta la simulacion. -->
+  <xacro:if value="$(arg spawn_load)">
+    <xacro:property name="_load_r" value="$(arg load_radius)"/>
+    <xacro:property name="_load_h" value="$(arg load_height)"/>
+    <xacro:property name="_load_m" value="$(arg load_mass)"/>
+    <xacro:property name="_load_x" value="$(arg load_x_offset)"/>
+    <link name="$(arg prefix)load_link">
+      <visual>
+        <origin xyz="0 0 0" rpy="${pi/2} 0 0"/>
+        <geometry>
+          <cylinder radius="${_load_r}" length="${_load_h}"/>
+        </geometry>
+        <material name="gold">
+          <color rgba="1.0 0.843 0.0 1.0"/>
+        </material>
+      </visual>
+      <collision>
+        <origin xyz="0 0 0" rpy="${pi/2} 0 0"/>
+        <geometry>
+          <cylinder radius="${_load_r}" length="${_load_h}"/>
+        </geometry>
+      </collision>
+      <inertial>
+        <origin xyz="0 0 0" rpy="0 0 0"/>
+        <mass value="${_load_m}"/>
+        <inertia
+          ixx="${_load_m * (3*_load_r*_load_r + _load_h*_load_h) / 12}"
+          iyy="${_load_m * _load_r * _load_r / 2}"
+          izz="${_load_m * (3*_load_r*_load_r + _load_h*_load_h) / 12}"
+          ixy="0" ixz="0" iyz="0"/>
+      </inertial>
+    </link>
+    <joint name="$(arg prefix)load_joint" type="fixed">
+      <parent link="$(arg prefix)end_effector_link"/>
+      <child  link="$(arg prefix)load_link"/>
+      <origin xyz="${_load_x} 0 0" rpy="0 0 0"/>
+    </joint>
+    <!-- Color dorado Ogre2 para Gazebo Fortress -->
+    <gazebo reference="$(arg prefix)load_link">
+      <visual>
+        <material>
+          <ambient>1.0 0.843 0.0 1</ambient>
+          <diffuse>1.0 0.843 0.0 1</diffuse>
+          <specular>0.5 0.420 0.0 1</specular>
+        </material>
+      </visual>
+    </gazebo>
+  </xacro:if>
 </robot>
