Commit message: Migrate simulation from Gazebo Classic to Gazebo Fortress
- Replace gazebo_ros2_control/GazeboSystem with gz_ros2_control/GazeboSimSystem
- Replace libgazebo_ros2_control.so plugin with gz_ros2_control-system
- Remove position workaround in arm joints (GazeboSimSystem supports pure effort)
- Replace gazebo.launch.py / spawn_entity.py with gz_sim.launch.py / ros_gz_sim create
- Add /clock bridge (ros_gz_bridge) required for use_sim_time with Fortress
- Add worlds/empty_world_fortress.sdf (SDF 1.9, inline ground_plane, no Fuel dependency)
- Update package.xml: gazebo_ros/gazebo_ros2_control → ros_gz_sim/ros_gz_bridge/gz_ros2_control
- Add worlds/ to CMakeLists.txt install(DIRECTORY ...) list

Co-Authored-By: Claude Sonnet 4.6 <noreply@anthropic.com>

File: xacro/open_manipulator_x_effort.ros2_control.xacro (robot description, xacro)
@@ -1,13 +1,9 @@
 <?xml version="1.0"?>
 <!--
-  ros2_control exclusivo para simulacion Gazebo con command_interface effort.
+  ros2_control exclusivo para simulacion Gazebo Fortress con command_interface effort.
   ADVERTENCIA: No compatible con hardware real Dynamixel.
-  NOTA IMPORTANTE sobre GazeboSystem 0.4.x:
-  GazeboSystem requiere command_interface "position" en cada joint durante
-  configureSim(). Sin el, falla la inicializacion y el controller_manager
-  nunca arranca (aunque el robot si aparece en Gazebo).
-  Por eso se declara "position" junto a "effort". En runtime, solo
-  arm_effort_controller reclamara "effort"; "position" queda disponible
-  pero sin controlador asignado, por lo que GazeboSystem lo ignora.
+  Usa gz_ros2_control/GazeboSimSystem (Gazebo Fortress / Ignition Gazebo 6).
+  GazeboSimSystem soporta effort puro sin necesidad del workaround de "position"
+  que requeria gazebo_ros2_control/GazeboSystem 0.4.x.
 -->
 <robot xmlns:xacro="http://www.ros.org/wiki/xacro">
@@ -15,8 +11,7 @@
     <ros2_control name="${name}" type="system">
       <hardware>
-        <plugin>gazebo_ros2_control/GazeboSystem</plugin>
+        <plugin>gz_ros2_control/GazeboSimSystem</plugin>
       </hardware>
       <joint name="${prefix}joint1">
-        <command_interface name="position"/>
         <command_interface name="effort">
           <param name="min">-1.0</param>
@@ -28,5 +23,4 @@
       </joint>
       <joint name="${prefix}joint2">
-        <command_interface name="position"/>
         <command_interface name="effort">
           <param name="min">-1.0</param>
@@ -38,5 +32,4 @@
       </joint>
       <joint name="${prefix}joint3">
-        <command_interface name="position"/>
         <command_interface name="effort">
           <param name="min">-1.0</param>
@@ -48,5 +41,4 @@
       </joint>
       <joint name="${prefix}joint4">
-        <command_interface name="position"/>
         <command_interface name="effort">
           <param name="min">-1.0</param>

File: xacro/open_manipulator_x_effort_robot.urdf.xacro (robot description, xacro)
@@ -4,5 +4,5 @@
   Reutiliza la cinematica y meshes del paquete original de ROBOTIS,
   pero sustituye el ros2_control xacro original por el de esfuerzo.
-  El plugin gazebo_ros2_control apunta al YAML de controladores de esfuerzo.
+  El plugin gz_ros2_control apunta al YAML de controladores de esfuerzo.
 -->
 <robot name="open_manipulator_x" xmlns:xacro="http://ros.org/wiki/xacro">
@@ -25,7 +25,8 @@
     name="OpenManipulatorXEffort"
     prefix="$(arg prefix)" />
-  <!-- Plugin gazebo_ros2_control apunta al YAML separado de controladores de esfuerzo -->
+  <!-- Plugin gz_ros2_control para Gazebo Fortress apunta al YAML de controladores -->
   <gazebo>
-    <plugin name="gazebo_ros2_control" filename="libgazebo_ros2_control.so">
+    <plugin filename="gz_ros2_control-system"
+            name="gz_ros2_control::GazeboSimROS2ControlPlugin">
       <parameters>$(find open_manipulator_x_torque_control)/config/effort_controllers.yaml</parameters>
     </plugin>
@@ -59,8 +60,7 @@
     </inertial>
   </link>
-  <!-- Material y colision Gazebo para la placa.
+  <!-- Propiedades de contacto Gazebo para la placa.
        self_collide permite que el brazo colisione con la placa (intra-modelo).
-       ODE ignora contactos entre links estaticos, por lo que link1 y la placa
-       no generan inestabilidad aunque esten en contacto. -->
+       Nota: material Gazebo/White eliminado — no existe en Ogre2 (Fortress). -->
   <gazebo reference="base_plate_02_link">
     <kp>1000000.0</kp>
@@ -69,5 +69,4 @@
     <mu2>0.6</mu2>
     <self_collide>true</self_collide>
-    <material>Gazebo/White</material>
   </gazebo>
   <!-- Placa anclada directamente al mundo. Ambos joints van a world para que

Commit message: Lab 5 TV-LQR: trajectory optimization, Riccati ZOH, Gazebo init config
- lab5_act1_sol.m: nueva solucion TV-LQR con joint limits, Riccati discreto ZOH,
  exportacion de figuras PNG/EPS y metricas de seguimiento
- Lab5_Export_Refs.m: Riccati continuo sqrt reemplazado por recursion discreta ZOH
  (garantiza S>0), Rk=100 para evitar singularidad
- gz_tvlqr_node / hw_tvlqr_node: eliminado 'lab5' de nombre ejecutable y nodo ROS;
  ruta CSV corregida a data/lab5/sim; fase warmup de compensacion gravitatoria
- xacro effort.ros2_control: posicion inicial configurable via sim_init_config.yaml
  usando xacro:if/unless con discretizacion ZOH correcta
- config/sim_init_config.yaml: nuevo archivo para elegir modo de inicio en Gazebo
  (equilibrio gravedad vs posicion articular fija)
- torque_sim.launch.py: lee sim_init_config.yaml y pasa args al xacro
- references/: trayectoria TV-LQR actualizada (N=30, Ts=0.05, x0->yf Lab5 Act.1)

Co-Authored-By: Claude Sonnet 4.6 <noreply@anthropic.com>

File: xacro/open_manipulator_x_effort.ros2_control.xacro (robot description, xacro)
@@ -6,11 +6,26 @@
   GazeboSimSystem soporta effort puro sin necesidad del workaround de "position"
   que requeria gazebo_ros2_control/GazeboSystem 0.4.x.
+  Parametros del macro:
+    use_fixed_init  True|False   — si True, aplica initial_value en cada joint
+    q1_init .. q4_init  [rad]   — posiciones iniciales (solo si use_fixed_init=True)
+  Notas de implementacion:
+    - El default debe ser el booleano Python False (no la cadena 'false'),
+      porque xacro convierte 'false' a False pero 'false'!='true' falla en
+      la comparacion == al recibir el bool True desde xacro:arg.
+    - xacro:if debe envolver bloques completos de state_interface, no
+      solo el param interno (limitacion del parser xacro).
+    - Condicion: ${use_fixed_init} — truthy check directo sobre el bool Python.
 -->
 <robot xmlns:xacro="http://www.ros.org/wiki/xacro">
-  <xacro:macro name="open_manipulator_x_effort_system" params="name prefix">
+  <xacro:macro name="open_manipulator_x_effort_system"
+               params="name prefix
+                       use_fixed_init:=False
+                       q1_init:=0.0  q2_init:=0.0
+                       q3_init:=0.0  q4_init:=0.0">
     <ros2_control name="${name}" type="system">
       <hardware>
         <plugin>gz_ros2_control/GazeboSimSystem</plugin>
       </hardware>
+      <!-- ── joint1 ────────────────────────────────────────────────────── -->
       <joint name="${prefix}joint1">
         <command_interface name="effort">
@@ -18,8 +33,19 @@
           <param name="max"> 1.0</param>
         </command_interface>
-        <state_interface name="position"/>
-        <state_interface name="velocity"/>
+        <xacro:if value="${use_fixed_init}">
+          <state_interface name="position">
+            <param name="initial_value">${q1_init}</param>
+          </state_interface>
+          <state_interface name="velocity">
+            <param name="initial_value">0.0</param>
+          </state_interface>
+        </xacro:if>
+        <xacro:unless value="${use_fixed_init}">
+          <state_interface name="position"/>
+          <state_interface name="velocity"/>
+        </xacro:unless>
         <state_interface name="effort"/>
       </joint>
+      <!-- ── joint2 ────────────────────────────────────────────────────── -->
       <joint name="${prefix}joint2">
         <command_interface name="effort">
@@ -27,8 +53,19 @@
           <param name="max"> 1.0</param>
         </command_interface>
-        <state_interface name="position"/>
-        <state_interface name="velocity"/>
+        <xacro:if value="${use_fixed_init}">
+          <state_interface name="position">
+            <param name="initial_value">${q2_init}</param>
+          </state_interface>
+          <state_interface name="velocity">
+            <param name="initial_value">0.0</param>
+          </state_interface>
+        </xacro:if>
+        <xacro:unless value="${use_fixed_init}">
+          <state_interface name="position"/>
+          <state_interface name="velocity"/>
+        </xacro:unless>
         <state_interface name="effort"/>
       </joint>
+      <!-- ── joint3 ────────────────────────────────────────────────────── -->
       <joint name="${prefix}joint3">
         <command_interface name="effort">
@@ -36,8 +73,19 @@
           <param name="max"> 1.0</param>
         </command_interface>
-        <state_interface name="position"/>
-        <state_interface name="velocity"/>
+        <xacro:if value="${use_fixed_init}">
+          <state_interface name="position">
+            <param name="initial_value">${q3_init}</param>
+          </state_interface>
+          <state_interface name="velocity">
+            <param name="initial_value">0.0</param>
+          </state_interface>
+        </xacro:if>
+        <xacro:unless value="${use_fixed_init}">
+          <state_interface name="position"/>
+          <state_interface name="velocity"/>
+        </xacro:unless>
         <state_interface name="effort"/>
       </joint>
+      <!-- ── joint4 ────────────────────────────────────────────────────── -->
       <joint name="${prefix}joint4">
         <command_interface name="effort">
@@ -45,9 +93,19 @@
           <param name="max"> 1.0</param>
         </command_interface>
-        <state_interface name="position"/>
-        <state_interface name="velocity"/>
+        <xacro:if value="${use_fixed_init}">
+          <state_interface name="position">
+            <param name="initial_value">${q4_init}</param>
+          </state_interface>
+          <state_interface name="velocity">
+            <param name="initial_value">0.0</param>
+          </state_interface>
+        </xacro:if>
+        <xacro:unless value="${use_fixed_init}">
+          <state_interface name="position"/>
+          <state_interface name="velocity"/>
+        </xacro:unless>
         <state_interface name="effort"/>
       </joint>
-      <!-- Gripper: solo control de posicion -->
+      <!-- ── Gripper: solo control de posicion ─────────────────────────── -->
       <joint name="${prefix}gripper_left_joint">
         <command_interface name="position"/>

File: xacro/open_manipulator_x_effort_robot.urdf.xacro (robot description, xacro)
@@ -7,6 +7,12 @@
 -->
 <robot name="open_manipulator_x" xmlns:xacro="http://ros.org/wiki/xacro">
-  <xacro:arg name="prefix"  default="" />
-  <xacro:arg name="use_sim" default="true" />
+  <xacro:arg name="prefix"         default="" />
+  <xacro:arg name="use_sim"        default="true" />
+  <!-- Posicion inicial: leida desde config/sim_init_config.yaml via launch file -->
+  <xacro:arg name="use_fixed_init" default="false" />
+  <xacro:arg name="q1_init"        default="0.0" />
+  <xacro:arg name="q2_init"        default="0.0" />
+  <xacro:arg name="q3_init"        default="0.0" />
+  <xacro:arg name="q4_init"        default="0.0" />
   <!-- Recursos graficos: colores Rviz y materiales Gazebo del paquete original -->
   <xacro:include filename="$(find open_manipulator_x_description)/gazebo/materials.xacro" />
@@ -24,5 +30,10 @@
   <xacro:open_manipulator_x_effort_system
     name="OpenManipulatorXEffort"
-    prefix="$(arg prefix)" />
+    prefix="$(arg prefix)"
+    use_fixed_init="$(arg use_fixed_init)"
+    q1_init="$(arg q1_init)"
+    q2_init="$(arg q2_init)"
+    q3_init="$(arg q3_init)"
+    q4_init="$(arg q4_init)" />
   <!-- Plugin gz_ros2_control para Gazebo Fortress apunta al YAML de controladores -->
   <gazebo>

Commit message: Carga en el efector: agarre por el diametro + re-sintonia del bloque theta_load
La carga cilindrica ahora se ve sostenida como en el robot real:
- Cilindro con eje a lo largo del eje Z del efector (caras arriba/abajo):
  el gripper lo toma alrededor de su DIAMETRO, no por las caras planas.
  Inercia recalculada para eje Z (Izz = m*r^2/2).
- Apertura automatica del gripper: el launch calcula
  gripper_init = load_radius - 0.021 (separacion entre dedos = 2r, limites
  del joint [-0.010, 0.019] → radios agarrables 11-40 mm) y lo inyecta como
  initial_value de los joints del gripper en el ros2_control; el
  GripperActionController mantiene la posicion sin necesidad de goal.
- Carga actual: 125 g, Ø38x13 mm, centrada en el EE (offset 0) →
  theta_load verdadero = [0.125, 0.125*0.126, 0, 0] = [0.125, 0.0158, 0, 0]
  documentado en yaml, nodo y LOAD_TRUE del script MATLAB.

Re-sintonia del bloque de carga del MRAC 12p (evidencia test 14: dm/dmcx
oscilaban en contrafase entre sus topes sobre la cresta mal condicionada de
las columnas m/mcx casi colineales, convergencia 0.2 s demasiado caliente):
- Gamma_dm 0.3 -> 0.05, Gamma_dmc 0.01 -> 0.002 (convergencia ~2-3 s
  amortiguada)
- sigma-modification ahora POR BLOQUE: 0.02 en theta_load (su prior es cero
  y la fuga fuerte peleaba contra el valor verdadero), 0.1 en el resto.

Co-Authored-By: Claude Fable 5 <noreply@anthropic.com>

File: xacro/open_manipulator_x_effort.ros2_control.xacro (robot description, xacro)
@@ -9,4 +9,8 @@
     use_fixed_init  True|False   — si True, aplica initial_value en cada joint
     q1_init .. q4_init  [rad]   — posiciones iniciales (solo si use_fixed_init=True)
+    gripper_init        [m]     — apertura inicial de cada dedo (incondicional;
+                                  separacion entre dedos = 0.042 + 2*gripper_init).
+                                  El GripperActionController mantiene esta
+                                  posicion mientras no reciba un goal.
   Notas de implementacion:
     - El default debe ser el booleano Python False (no la cadena 'false'),
@@ -22,5 +26,6 @@
                        use_fixed_init:=False
                        q1_init:=0.0  q2_init:=0.0
-                       q3_init:=0.0  q4_init:=0.0">
+                       q3_init:=0.0  q4_init:=0.0
+                       gripper_init:=0.0">
     <ros2_control name="${name}" type="system">
       <hardware>
@@ -108,7 +113,12 @@
       </joint>
       <!-- ── Gripper: solo control de posicion ─────────────────────────── -->
+      <!-- initial_value abre los dedos a la medida de la carga (tangentes al
+           diametro del cilindro); gz_ros2_control inicializa el comando de
+           posicion con este valor y lo mantiene sin necesidad de goal. -->
       <joint name="${prefix}gripper_left_joint">
         <command_interface name="position"/>
-        <state_interface name="position"/>
+        <state_interface name="position">
+          <param name="initial_value">${gripper_init}</param>
+        </state_interface>
         <state_interface name="velocity"/>
         <state_interface name="effort"/>
@@ -118,5 +128,7 @@
         <param name="multiplier">1</param>
         <command_interface name="position"/>
-        <state_interface name="position"/>
+        <state_interface name="position">
+          <param name="initial_value">${gripper_init}</param>
+        </state_interface>
         <state_interface name="velocity"/>
         <state_interface name="effort"/>

File: xacro/open_manipulator_x_effort_robot.urdf.xacro (robot description, xacro)
@@ -25,4 +25,8 @@
   <xacro:arg name="load_mass"     default="0.1"   />   <!-- masa          [kg] -->
   <xacro:arg name="load_x_offset" default="0.0"   />   <!-- offset en X   [m] -->
+  <!-- Apertura inicial del gripper [m/joint]: el launch la calcula como
+       load_radius - 0.021 para que los dedos queden tangentes al diametro
+       de la carga (separacion entre origenes de dedos = 0.042 + 2*valor). -->
+  <xacro:arg name="gripper_init"  default="0.0"   />
   <!-- Recursos graficos: colores Rviz y materiales Gazebo del paquete original -->
   <xacro:include filename="$(find open_manipulator_x_description)/gazebo/materials.xacro" />
@@ -50,5 +54,6 @@
     q2_init="$(arg q2_init)"
     q3_init="$(arg q3_init)"
-    q4_init="$(arg q4_init)" />
+    q4_init="$(arg q4_init)"
+    gripper_init="$(arg gripper_init)" />
   <!-- Plugin gz_ros2_control para Gazebo Fortress apunta al YAML de controladores -->
   <gazebo>
@@ -146,9 +151,12 @@
   </joint>
   <!-- ── Carga cilindrica en el efector final ──────────────────────────────────
-       Cilindro solido cuyo eje coincide con el eje Y de end_effector_link.
-       Las caras circulares apuntan en +Y / -Y (rpy pi/2 0 0 alinea eje Z→Y).
-       Inercia de cilindro solido con eje a lo largo de Y:
-         Ixx = Izz = m*(3r^2 + h^2)/12
-         Iyy = m*r^2/2
+       Cilindro solido cuyo eje coincide con el eje Z de end_effector_link
+       (rpy 0 0 0: el eje del primitivo <cylinder> ya es Z). Las caras planas
+       apuntan arriba/abajo y el gripper lo sostiene alrededor de su DIAMETRO
+       (dedos tangentes a la superficie lateral, separacion 2r fijada por
+       gripper_init en el launch), como el robot real.
+       Inercia de cilindro solido con eje a lo largo de Z:
+         Ixx = Iyy = m*(3r^2 + h^2)/12
+         Izz = m*r^2/2
        Solo se instancia si spawn_load:=true; en caso contrario no existe en
        el arbol cinematico y no afecta la simulacion. -->
@@ -160,5 +168,5 @@
     <link name="$(arg prefix)load_link">
       <visual>
-        <origin xyz="0 0 0" rpy="${pi/2} 0 0"/>
+        <origin xyz="0 0 0" rpy="0 0 0"/>
         <geometry>
           <cylinder radius="${_load_r}" length="${_load_h}"/>
@@ -169,5 +177,5 @@
       </visual>
       <collision>
-        <origin xyz="0 0 0" rpy="${pi/2} 0 0"/>
+        <origin xyz="0 0 0" rpy="0 0 0"/>
         <geometry>
           <cylinder radius="${_load_r}" length="${_load_h}"/>
@@ -179,6 +187,6 @@
         <inertia
           ixx="${_load_m * (3*_load_r*_load_r + _load_h*_load_h) / 12}"
-          iyy="${_load_m * _load_r * _load_r / 2}"
-          izz="${_load_m * (3*_load_r*_load_r + _load_h*_load_h) / 12}"
+          iyy="${_load_m * (3*_load_r*_load_r + _load_h*_load_h) / 12}"
+          izz="${_load_m * _load_r * _load_r / 2}"
           ixy="0" ixz="0" iyz="0"/>
       </inertial>
