Commit message: Migrate control nodes to ROBOTIS-spec URDF and raise torque limits
Switch all control nodes from openmani.urdf to open_manipulator_x.urdf
(official ROBOTIS inertial parameters). Affects FL/IO instructor and
student nodes plus the gravity compensation nodes.

Raise TAU_MAX from 0.82/1.0 to 1.5 N.m across instructor and gravity
nodes, and add the torque-saturation logic to hw_fl_control_node
(mirroring gz_fl/gz_io/hw_io). The heavier link5 (143g->236g) pushes
G(q) on joint2 above 0.82 N.m, which saturated the old limit
permanently. Student template TAU_MAX placeholders are left as-is.

Update the effort ros2_control command_interface limits to +/-1.5 N.m
and the kinematic xacro joint effort limits to 1.5, matching TAU_MAX.

Add scripts/compare_urdf_dynamics.py to verify M(q)/G(q)/NLE coherence
between the old and new URDF (sign, structure, positive-definiteness).

Update plots_IO_control.m saturation reference lines to +/-1.5 N.m.

Co-Authored-By: Claude Opus 4.8 <noreply@anthropic.com>

File: xacro/open_manipulator_x.urdf.xacro (robot description, xacro)
@@ -51,5 +51,5 @@
       <origin xyz="0.012 0.0 0.017" rpy="0 0 0"/>
       <axis xyz="0 0 1"/>
-      <limit velocity="4.8" effort="1" lower="${-pi}" upper="${pi}" />
+      <limit velocity="4.8" effort="1.5" lower="${-pi}" upper="${pi}" />
       <dynamics damping="0.1"/>
     </joint>
@@ -83,5 +83,5 @@
       <origin xyz="0.0 0.0 0.0595" rpy="0 0 0"/>
       <axis xyz="0 1 0"/>
-      <limit velocity="4.8" effort="1" lower="${-1.5}" upper="${1.5}" />
+      <limit velocity="4.8" effort="1.5" lower="${-1.5}" upper="${1.5}" />
       <dynamics damping="0.1"/>
     </joint>
@@ -115,5 +115,5 @@
       <origin xyz="0.024 0 0.128" rpy="0 0 0"/>
       <axis xyz="0 1 0"/>
-      <limit velocity="4.8" effort="1" lower="${-1.5}" upper="${1.4}" />
+      <limit velocity="4.8" effort="1.5" lower="${-1.5}" upper="${1.4}" />
       <dynamics damping="0.1"/>
     </joint>
@@ -148,5 +148,5 @@
       <origin xyz="0.124 0.0 0.0" rpy="0 0 0"/>
       <axis xyz="0 1 0"/>
-      <limit velocity="4.8" effort="1" lower="${-1.7}" upper="${1.97}" />
+      <limit velocity="4.8" effort="1.5" lower="${-1.7}" upper="${1.97}" />
       <dynamics damping="0.1"/>
     </joint>

File: xacro/open_manipulator_x_effort.ros2_control.xacro (robot description, xacro)
@@ -30,6 +30,6 @@
       <joint name="${prefix}joint1">
         <command_interface name="effort">
-          <param name="min">-1.0</param>
-          <param name="max"> 1.0</param>
+          <param name="min">-1.5</param>
+          <param name="max"> 1.5</param>
         </command_interface>
         <xacro:if value="${use_fixed_init}">
@@ -50,6 +50,6 @@
       <joint name="${prefix}joint2">
         <command_interface name="effort">
-          <param name="min">-1.0</param>
-          <param name="max"> 1.0</param>
+          <param name="min">-1.5</param>
+          <param name="max"> 1.5</param>
         </command_interface>
         <xacro:if value="${use_fixed_init}">
@@ -70,6 +70,6 @@
       <joint name="${prefix}joint3">
         <command_interface name="effort">
-          <param name="min">-1.0</param>
-          <param name="max"> 1.0</param>
+          <param name="min">-1.5</param>
+          <param name="max"> 1.5</param>
         </command_interface>
         <xacro:if value="${use_fixed_init}">
@@ -90,6 +90,6 @@
       <joint name="${prefix}joint4">
         <command_interface name="effort">
-          <param name="min">-1.0</param>
-          <param name="max"> 1.0</param>
+          <param name="min">-1.5</param>
+          <param name="max"> 1.5</param>
         </command_interface>
         <xacro:if value="${use_fixed_init}">

Commit message: URDF/Xacro: update joint dynamics with identified friction parameters
Replace generic damping=0.1 with OLS-identified values from motor_params.yaml
(Fv→damping, Fc→friction, converted via kt=1.654 N·m/A, Iu=0.00269 A/tick):
  J1: damping=0.0230  friction=0.0168
  J2: damping=0.0194  friction=0.0089
  J3: damping=0.0229  friction=0.0094
  J4: damping=0.0158  friction=0.0377
Gripper joints unchanged.

Co-Authored-By: Claude Sonnet 4.6 <noreply@anthropic.com>

File: xacro/open_manipulator_x.urdf.xacro (robot description, xacro)
@@ -49,5 +49,5 @@
       <axis xyz="0 0 1"/>
       <limit velocity="4.8" effort="1.5" lower="${-3*pi/4}" upper="${3*pi/4}" />
-      <dynamics damping="0.1"/>
+      <dynamics damping="0.0230" friction="0.0168"/>
     </joint>
     <link name="${prefix}link2">
@@ -80,5 +80,5 @@
       <axis xyz="0 1 0"/>
       <limit velocity="4.8" effort="1.5" lower="${-11*pi/18}" upper="${5*pi/9}" />
-      <dynamics damping="0.1"/>
+      <dynamics damping="0.0194" friction="0.0089"/>
     </joint>
     <link name="${prefix}link3">
@@ -111,5 +111,5 @@
       <axis xyz="0 1 0"/>
       <limit velocity="4.8" effort="1.5" lower="${-11*pi/18}" upper="${pi/2}" />
-      <dynamics damping="0.1"/>
+      <dynamics damping="0.0229" friction="0.0094"/>
     </joint>
     <link name="${prefix}link4">
@@ -142,5 +142,5 @@
       <axis xyz="0 1 0"/>
       <limit velocity="4.8" effort="1.5" lower="-1.8" upper="2.1" />
-      <dynamics damping="0.1"/>
+      <dynamics damping="0.0158" friction="0.0377"/>
     </joint>
     <link name="${prefix}link5">

Commit message: xacro: add mass_inertia_scale and friction_scale args to URDF
- open_manipulator_x.urdf.xacro: macro now accepts mass_inertia_scale
  and friction_scale params; applies them via xacro expressions to
  link1..link5 inertials and joint1..joint4 friction respectively.
  Gripper links, base plate, and damping values are not affected.
- open_manipulator_x_effort_robot.urdf.xacro: declares xacro:arg for
  both scales (default 1.0) and forwards them to the kinematic macro.
- torque_sim.launch.py: reads mass_inertia_scale and friction_scale
  from sim_init_config.yaml and passes them to the xacro command.
- sim_init_config.yaml: adds mass_inertia_scale and friction_scale
  entries (both default 1.0) with usage comments.

Co-Authored-By: Claude Sonnet 4.6 <noreply@anthropic.com>

File: xacro/open_manipulator_x.urdf.xacro (robot description, xacro)
@@ -9,4 +9,7 @@
     - joint4      : limites actualizados a [-1.8, 2.1] rad
     - gripper_right_joint: damping 0.1 -> 0.7 (igual que ROBOTIS URDF oficial)
+  Parametros de escala (configurables desde sim_init_config.yaml):
+    mass_inertia_scale : factor multiplicativo para masas e inercias de link1..link5
+    friction_scale     : factor multiplicativo para friccion de joint1..joint4
   Sin cambios:
     - Meshes (mismo paquete open_manipulator_x_description)
@@ -16,5 +19,6 @@
 -->
 <robot xmlns:xacro="http://www.ros.org/wiki/xacro">
-  <xacro:macro name="open_manipulator_x" params="prefix=''">
+  <xacro:macro name="open_manipulator_x"
+               params="prefix='' mass_inertia_scale='1.0' friction_scale='1.0'">
     <xacro:property
       name="meshes_file_direction"
@@ -37,8 +41,8 @@
       <inertial>
         <origin xyz="0.000308 0.000000 0.017927" rpy="0 0 0"/>
-        <mass value="0.0804" />
-        <inertia ixx="1.275713e-05" ixy="0.000000e+00" ixz="-1.794293e-07"
-                 iyy="2.234728e-05" iyz="0.000000e+00"
-                 izz="1.965878e-05" />
+        <mass value="${0.0804 * mass_inertia_scale}" />
+        <inertia ixx="${1.275713e-05 * mass_inertia_scale}" ixy="0.000000e+00" ixz="${-1.794293e-07 * mass_inertia_scale}"
+                 iyy="${2.234728e-05 * mass_inertia_scale}" iyz="0.000000e+00"
+                 izz="${1.965878e-05 * mass_inertia_scale}" />
       </inertial>
     </link>
@@ -49,5 +53,5 @@
       <axis xyz="0 0 1"/>
       <limit velocity="4.8" effort="1.5" lower="${-3*pi/4}" upper="${3*pi/4}" />
-      <dynamics damping="0.0230" friction="0.0168"/>
+      <dynamics damping="0.0230" friction="${0.0168 * friction_scale}"/>
     </joint>
     <link name="${prefix}link2">
@@ -68,8 +72,8 @@
       <inertial>
         <origin xyz="0.000000 0.000657 0.044319" rpy="0 0 0"/>
-        <mass value="0.0970" />
-        <inertia ixx="3.078317e-05" ixy="0.000000e+00" ixz="0.000000e+00"
-                 iyy="2.670366e-05" iyz="-1.289659e-07"
-                 izz="1.627175e-05" />
+        <mass value="${0.0970 * mass_inertia_scale}" />
+        <inertia ixx="${3.078317e-05 * mass_inertia_scale}" ixy="0.000000e+00" ixz="0.000000e+00"
+                 iyy="${2.670366e-05 * mass_inertia_scale}" iyz="${-1.289659e-07 * mass_inertia_scale}"
+                 izz="${1.627175e-05 * mass_inertia_scale}" />
       </inertial>
     </link>
@@ -80,5 +84,5 @@
       <axis xyz="0 1 0"/>
       <limit velocity="4.8" effort="1.5" lower="${-11*pi/18}" upper="${5*pi/9}" />
-      <dynamics damping="0.0194" friction="0.0089"/>
+      <dynamics damping="0.0194" friction="${0.0089 * friction_scale}"/>
     </joint>
     <link name="${prefix}link3">
@@ -99,8 +103,8 @@
       <inertial>
         <origin xyz="0.007606 0.000389 0.099924" rpy="0 0 0"/>
-        <mass value="0.1235" />
-        <inertia ixx="1.979680e-04" ixy="-2.511443e-07" ixz="-2.497601e-05"
-                 iyy="2.046627e-04" iyz="-1.351040e-06"
-                 izz="3.374865e-05" />
+        <mass value="${0.1235 * mass_inertia_scale}" />
+        <inertia ixx="${1.979680e-04 * mass_inertia_scale}" ixy="${-2.511443e-07 * mass_inertia_scale}" ixz="${-2.497601e-05 * mass_inertia_scale}"
+                 iyy="${2.046627e-04 * mass_inertia_scale}" iyz="${-1.351040e-06 * mass_inertia_scale}"
+                 izz="${3.374865e-05 * mass_inertia_scale}" />
       </inertial>
     </link>
@@ -111,5 +115,5 @@
       <axis xyz="0 1 0"/>
       <limit velocity="4.8" effort="1.5" lower="${-11*pi/18}" upper="${pi/2}" />
-      <dynamics damping="0.0229" friction="0.0094"/>
+      <dynamics damping="0.0229" friction="${0.0094 * friction_scale}"/>
     </joint>
     <link name="${prefix}link4">
@@ -130,8 +134,8 @@
       <inertial>
         <origin xyz="0.089168 0.000437 0.000001" rpy="0 0 0"/>
-        <mass value="0.1151" />
-        <inertia ixx="1.930305e-05" ixy="-1.189078e-06" ixz="3.461654e-09"
-                 iyy="1.483284e-04" iyz="0.000000e+00"
-                 izz="1.547550e-04" />
+        <mass value="${0.1151 * mass_inertia_scale}" />
+        <inertia ixx="${1.930305e-05 * mass_inertia_scale}" ixy="${-1.189078e-06 * mass_inertia_scale}" ixz="${3.461654e-09 * mass_inertia_scale}"
+                 iyy="${1.483284e-04 * mass_inertia_scale}" iyz="0.000000e+00"
+                 izz="${1.547550e-04 * mass_inertia_scale}" />
       </inertial>
     </link>
@@ -142,5 +146,5 @@
       <axis xyz="0 1 0"/>
       <limit velocity="4.8" effort="1.5" lower="-1.8" upper="2.1" />
-      <dynamics damping="0.0158" friction="0.0377"/>
+      <dynamics damping="0.0158" friction="${0.0377 * friction_scale}"/>
     </joint>
     <link name="${prefix}link5">
@@ -161,8 +165,8 @@
       <inertial>
         <origin xyz="0.062451 0.000000 0.005878" rpy="0 0 0"/>
-        <mass value="0.2206" />
-        <inertia ixx="1.344328e-04" ixy="-1.788649e-08" ixz="2.259163e-05"
-                 iyy="1.892619e-04" iyz="9.936937e-07"
-                 izz="2.174510e-04" />
+        <mass value="${0.2206 * mass_inertia_scale}" />
+        <inertia ixx="${1.344328e-04 * mass_inertia_scale}" ixy="${-1.788649e-08 * mass_inertia_scale}" ixz="${2.259163e-05 * mass_inertia_scale}"
+                 iyy="${1.892619e-04 * mass_inertia_scale}" iyz="${9.936937e-07 * mass_inertia_scale}"
+                 izz="${2.174510e-04 * mass_inertia_scale}" />
       </inertial>
     </link>

File: xacro/open_manipulator_x_effort_robot.urdf.xacro (robot description, xacro)
@@ -15,4 +15,7 @@
   <xacro:arg name="q3_init"        default="0.0" />
   <xacro:arg name="q4_init"        default="0.0" />
+  <!-- Escalas de dinamica: leidas desde config/sim_init_config.yaml via launch file -->
+  <xacro:arg name="mass_inertia_scale" default="1.0" />
+  <xacro:arg name="friction_scale"     default="1.0" />
   <!-- Recursos graficos: colores Rviz y materiales Gazebo del paquete original -->
   <xacro:include filename="$(find open_manipulator_x_description)/gazebo/materials.xacro" />
@@ -26,5 +29,7 @@
   <xacro:include filename="$(find open_manipulator_x_torque_control)/xacro/open_manipulator_x_effort.ros2_control.xacro" />
   <!-- Instanciar cadena cinematica -->
-  <xacro:open_manipulator_x prefix="$(arg prefix)" />
+  <xacro:open_manipulator_x prefix="$(arg prefix)"
+                             mass_inertia_scale="$(arg mass_inertia_scale)"
+                             friction_scale="$(arg friction_scale)" />
   <!-- Instanciar propiedades Gazebo -->
   <xacro:open_manipulator_x_gazebo prefix="$(arg prefix)" />

Commit message: xacro/config: rename friction_scale → damping_scale, apply to damping only
El parametro friction_scale escalaba la friccion de joint1..4; ahora
damping_scale escala el damping viscoso y la friccion queda fija con
sus valores nominales identificados.

Archivos afectados:
  xacro/open_manipulator_x.urdf.xacro               — param + 4 joints
  xacro/open_manipulator_x_effort_robot.urdf.xacro  — xacro:arg + instancia
  config/sim_init_config.yaml                        — clave + comentarios
  launch/torque_sim.launch.py                        — lectura YAML + pase al xacro

Co-Authored-By: Claude Sonnet 4.6 <noreply@anthropic.com>

File: xacro/open_manipulator_x.urdf.xacro (robot description, xacro)
@@ -11,5 +11,5 @@
   Parametros de escala (configurables desde sim_init_config.yaml):
     mass_inertia_scale : factor multiplicativo para masas e inercias de link1..link5
-    friction_scale     : factor multiplicativo para friccion de joint1..joint4
+    damping_scale      : factor multiplicativo para damping de joint1..joint4 (friction fijo)
   Sin cambios:
     - Meshes (mismo paquete open_manipulator_x_description)
@@ -20,5 +20,5 @@
 <robot xmlns:xacro="http://www.ros.org/wiki/xacro">
   <xacro:macro name="open_manipulator_x"
-               params="prefix='' mass_inertia_scale='1.0' friction_scale='1.0'">
+               params="prefix='' mass_inertia_scale='1.0' damping_scale='1.0'">
     <xacro:property
       name="meshes_file_direction"
@@ -53,5 +53,5 @@
       <axis xyz="0 0 1"/>
       <limit velocity="4.8" effort="1.5" lower="${-3*pi/4}" upper="${3*pi/4}" />
-      <dynamics damping="0.0230" friction="${0.0168 * friction_scale}"/>
+      <dynamics damping="${0.0230 * damping_scale}" friction="0.0168"/>
     </joint>
     <link name="${prefix}link2">
@@ -84,5 +84,5 @@
       <axis xyz="0 1 0"/>
       <limit velocity="4.8" effort="1.5" lower="${-11*pi/18}" upper="${5*pi/9}" />
-      <dynamics damping="0.0194" friction="${0.0089 * friction_scale}"/>
+      <dynamics damping="${0.0194 * damping_scale}" friction="0.0089"/>
     </joint>
     <link name="${prefix}link3">
@@ -115,5 +115,5 @@
       <axis xyz="0 1 0"/>
       <limit velocity="4.8" effort="1.5" lower="${-11*pi/18}" upper="${pi/2}" />
-      <dynamics damping="0.0229" friction="${0.0094 * friction_scale}"/>
+      <dynamics damping="${0.0229 * damping_scale}" friction="0.0094"/>
     </joint>
     <link name="${prefix}link4">
@@ -146,5 +146,5 @@
       <axis xyz="0 1 0"/>
       <limit velocity="4.8" effort="1.5" lower="-1.8" upper="2.1" />
-      <dynamics damping="0.0158" friction="${0.0377 * friction_scale}"/>
+      <dynamics damping="${0.0158 * damping_scale}" friction="0.0377"/>
     </joint>
     <link name="${prefix}link5">

File: xacro/open_manipulator_x_effort_robot.urdf.xacro (robot description, xacro)
@@ -17,5 +17,5 @@
   <!-- Escalas de dinamica: leidas desde config/sim_init_config.yaml via launch file -->
   <xacro:arg name="mass_inertia_scale" default="1.0" />
-  <xacro:arg name="friction_scale"     default="1.0" />
+  <xacro:arg name="damping_scale"      default="1.0" />
   <!-- Recursos graficos: colores Rviz y materiales Gazebo del paquete original -->
   <xacro:include filename="$(find open_manipulator_x_description)/gazebo/materials.xacro" />
@@ -31,5 +31,5 @@
   <xacro:open_manipulator_x prefix="$(arg prefix)"
                              mass_inertia_scale="$(arg mass_inertia_scale)"
-                             friction_scale="$(arg friction_scale)" />
+                             damping_scale="$(arg damping_scale)" />
   <!-- Instanciar propiedades Gazebo -->
   <xacro:open_manipulator_x_gazebo prefix="$(arg prefix)" />

Commit message: xacro/sim: add independent friction_scale for joint1..4 friction
Parametro friction_scale configurable desde sim_init_config.yaml que
escala el parametro friction de joint1..joint4 de forma independiente
a damping_scale. Permite simular desde friccion nula hasta mayor que la
nominal sin afectar el damping viscoso.

  friction_scale: 0.0  → sin friccion de Coulomb
  friction_scale: 1.0  → valores nominales identificados
  friction_scale: >1   → mayor friccion

Archivos: xacro/open_manipulator_x.urdf.xacro (macro param + 4 joints)
          xacro/open_manipulator_x_effort_robot.urdf.xacro (arg + instancia)
          config/sim_init_config.yaml
          launch/torque_sim.launch.py

Co-Authored-By: Claude Sonnet 4.6 <noreply@anthropic.com>

File: xacro/open_manipulator_x.urdf.xacro (robot description, xacro)
@@ -11,5 +11,6 @@
   Parametros de escala (configurables desde sim_init_config.yaml):
     mass_inertia_scale : factor multiplicativo para masas e inercias de link1..link5
-    damping_scale      : factor multiplicativo para damping de joint1..joint4 (friction fijo)
+    damping_scale      : factor multiplicativo para damping de joint1..joint4
+    friction_scale     : factor multiplicativo para friction de joint1..joint4
   Sin cambios:
     - Meshes (mismo paquete open_manipulator_x_description)
@@ -20,5 +21,5 @@
 <robot xmlns:xacro="http://www.ros.org/wiki/xacro">
   <xacro:macro name="open_manipulator_x"
-               params="prefix='' mass_inertia_scale='1.0' damping_scale='1.0'">
+               params="prefix='' mass_inertia_scale='1.0' damping_scale='1.0' friction_scale='1.0'">
     <xacro:property
       name="meshes_file_direction"
@@ -53,5 +54,5 @@
       <axis xyz="0 0 1"/>
       <limit velocity="4.8" effort="1.5" lower="${-3*pi/4}" upper="${3*pi/4}" />
-      <dynamics damping="${0.0230 * damping_scale}" friction="0.0168"/>
+      <dynamics damping="${0.0230 * damping_scale}" friction="${0.0168 * friction_scale}"/>
     </joint>
     <link name="${prefix}link2">
@@ -84,5 +85,5 @@
       <axis xyz="0 1 0"/>
       <limit velocity="4.8" effort="1.5" lower="${-11*pi/18}" upper="${5*pi/9}" />
-      <dynamics damping="${0.0194 * damping_scale}" friction="0.0089"/>
+      <dynamics damping="${0.0194 * damping_scale}" friction="${0.0089 * friction_scale}"/>
     </joint>
     <link name="${prefix}link3">
@@ -115,5 +116,5 @@
       <axis xyz="0 1 0"/>
       <limit velocity="4.8" effort="1.5" lower="${-11*pi/18}" upper="${pi/2}" />
-      <dynamics damping="${0.0229 * damping_scale}" friction="0.0094"/>
+      <dynamics damping="${0.0229 * damping_scale}" friction="${0.0094 * friction_scale}"/>
     </joint>
     <link name="${prefix}link4">
@@ -146,5 +147,5 @@
       <axis xyz="0 1 0"/>
       <limit velocity="4.8" effort="1.5" lower="-1.8" upper="2.1" />
-      <dynamics damping="${0.0158 * damping_scale}" friction="0.0377"/>
+      <dynamics damping="${0.0158 * damping_scale}" friction="${0.0377 * friction_scale}"/>
     </joint>
     <link name="${prefix}link5">

File: xacro/open_manipulator_x_effort_robot.urdf.xacro (robot description, xacro)
@@ -18,4 +18,5 @@
   <xacro:arg name="mass_inertia_scale" default="1.0" />
   <xacro:arg name="damping_scale"      default="1.0" />
+  <xacro:arg name="friction_scale"     default="1.0" />
   <!-- Carga cilindrica en el efector final: configurables desde sim_init_config.yaml -->
   <xacro:arg name="spawn_load"    default="false" />
@@ -37,5 +38,6 @@
   <xacro:open_manipulator_x prefix="$(arg prefix)"
                              mass_inertia_scale="$(arg mass_inertia_scale)"
-                             damping_scale="$(arg damping_scale)" />
+                             damping_scale="$(arg damping_scale)"
+                             friction_scale="$(arg friction_scale)" />
   <!-- Instanciar propiedades Gazebo -->
   <xacro:open_manipulator_x_gazebo prefix="$(arg prefix)" />

Commit message: urdf/xacro: update joint damping/friction from identified motor model
Convert the identified friction (motorXM430W350T_params.yaml, in current ticks)
to physical joint torque units:
  damping  = motor_Fv / motor_alpha   [N·m·s/rad]
  friction = motor_Fc / motor_alpha   [N·m]

J1..J4 damping: [0.0367, 0.0000, 0.0000, 0.0050]
J1..J4 friction:[0.0146, 0.0830, 0.1143, 0.0413]

J2/J3 viscous damping is ~0 (Coulomb-dominated per identification). xacro keeps
the damping_scale/friction_scale factors; gripper joints unchanged.

Co-Authored-By: Claude Opus 4.8 <noreply@anthropic.com>

File: xacro/open_manipulator_x.urdf.xacro (robot description, xacro)
@@ -54,5 +54,5 @@
       <axis xyz="0 0 1"/>
       <limit velocity="4.8" effort="1.5" lower="${-3*pi/4}" upper="${3*pi/4}" />
-      <dynamics damping="${0.0230 * damping_scale}" friction="${0.0168 * friction_scale}"/>
+      <dynamics damping="${0.0367 * damping_scale}" friction="${0.0146 * friction_scale}"/>
     </joint>
     <link name="${prefix}link2">
@@ -85,5 +85,5 @@
       <axis xyz="0 1 0"/>
       <limit velocity="4.8" effort="1.5" lower="${-11*pi/18}" upper="${5*pi/9}" />
-      <dynamics damping="${0.0194 * damping_scale}" friction="${0.0089 * friction_scale}"/>
+      <dynamics damping="${0.0000 * damping_scale}" friction="${0.0830 * friction_scale}"/>
     </joint>
     <link name="${prefix}link3">
@@ -116,5 +116,5 @@
       <axis xyz="0 1 0"/>
       <limit velocity="4.8" effort="1.5" lower="${-11*pi/18}" upper="${pi/2}" />
-      <dynamics damping="${0.0229 * damping_scale}" friction="${0.0094 * friction_scale}"/>
+      <dynamics damping="${0.0000 * damping_scale}" friction="${0.1143 * friction_scale}"/>
     </joint>
     <link name="${prefix}link4">
@@ -147,5 +147,5 @@
       <axis xyz="0 1 0"/>
       <limit velocity="4.8" effort="1.5" lower="-1.8" upper="2.1" />
-      <dynamics damping="${0.0158 * damping_scale}" friction="${0.0377 * friction_scale}"/>
+      <dynamics damping="${0.0050 * damping_scale}" friction="${0.0413 * friction_scale}"/>
     </joint>
     <link name="${prefix}link5">
