Commit message: urdf/xacro: actualizar inercias medidas y limites articulares
Propiedades inerciales de link1-link5 actualizadas con masas medidas
en balanza fisica y tensores de Inventor CAD escalados por m_real/m_CAD.
Limites de joint4 ajustados a [-1.8, 2.1] rad; joints 1-3 a ±3π/4,
-11π/18..5π/9, -11π/18..π/2. Cambios reflejados en URDF y xacro.

Co-Authored-By: Claude Sonnet 4.6 <noreply@anthropic.com>

File: urdf/open_manipulator_x.urdf (robot description, URDF)
Before this commit: robot open_manipulator, 8 links, 7 joints
Links:
- link link1: mass 7.9119962e-02 -> 0.0804
- link link2: mass 1.0483260e-01 -> 0.0970
- link link3: mass 1.4234630e-01 -> 0.1235
- link link4: mass 1.3467049e-01 -> 0.1151
- link link5: mass 2.3650927e-01 -> 0.2206
Joints:
- joint joint1: limit lower=-2.827433388230814 upper=2.827433388230814 effort=1 velocity=4.8 -> lower=-2.356194490192345 upper=2.356194490192345 effort=1 velocity=4.8
- joint joint2: limit lower=-1.790707812546182 upper=1.5707963267948966 effort=1 velocity=4.8 -> lower=-1.9198621771937625 upper=1.7453292519943295 effort=1 velocity=4.8
- joint joint3: limit lower=-0.9424777960769379 upper=1.382300767579509 effort=1 velocity=4.8 -> lower=-1.9198621771937625 upper=1.5707963267948966 effort=1 velocity=4.8
- joint joint4: limit lower=-1.790707812546182 upper=2.0420352248333655 effort=1 velocity=4.8 -> lower=-1.8 upper=2.1 effort=1 velocity=4.8

File: xacro/open_manipulator_x.urdf.xacro (robot description, xacro)
@@ -3,16 +3,13 @@
   open_manipulator_x.urdf.xacro
   Copia local de open_manipulator_x_description/urdf/open_manipulator_x.urdf.xacro
-  con propiedades inerciales actualizadas desde el e-Manual oficial de ROBOTIS
-  (platform-openmanipulator-x-specification.pdf, Section 2.3 Inertia).
+  con propiedades inerciales actualizadas desde mediciones reales de masa (balanza)
+  y tensores de inercia de Autodesk Inventor CAD escalados por m_real/m_CAD.
   Cambios respecto al original del paquete de descripcion:
-    - link2 : masa/CoG/tensor del Joint 1 del PDF  (R = I, sin rotacion de frame)
-    - link3 : masa/CoG/tensor del Joint 2 del PDF  (R = Rz(180 deg))
-    - link4 : masa/CoG/tensor del Joint 3 del PDF  (R = R_alt: Cz->URDF_x, Cx->+URDF_z)
-    - link5 : masa/CoG/tensor del Joint 4 del PDF  (R = R_alt: Cz->URDF_x, Cx->+URDF_z)
+    - link1-link5 : masa/CoG/tensor medidos fisicamente + Inventor (m_real/m_CAD)
+    - joint4      : limites actualizados a [-1.8, 2.1] rad
     - gripper_right_joint: damping 0.1 -> 0.7 (igual que ROBOTIS URDF oficial)
   Sin cambios:
-    - link1 inertial (sin contraparte en el PDF)
     - Meshes (mismo paquete open_manipulator_x_description)
-    - Origenes, ejes y limites articulares
+    - Origenes y ejes articulares
     - Gripper links inertial (masa dummy)
     - Estructura dummy_mimic_fix
@@ -37,11 +34,11 @@
         </geometry>
       </collision>
-      <!-- link1: sin contraparte en el PDF — valores del paquete de descripcion originales -->
-      <inertial>
-        <origin xyz="3.0876154e-04 0.0000000e+00 -1.2176461e-04" />
-        <mass value="7.9119962e-02" />
-        <inertia ixx="1.2505234e-05" ixy="0.0" ixz="-1.7855208e-07"
-                 iyy="2.1898364e-05" iyz="0.0"
-                 izz="1.9267361e-05" />
+      <!-- link1 — balanza + Inventor CAD (escalado m_real/m_CAD) -->
+      <inertial>
+        <origin xyz="0.000308 0.000000 0.017927" rpy="0 0 0"/>
+        <mass value="0.0804" />
+        <inertia ixx="1.275713e-05" ixy="0.000000e+00" ixz="-1.794293e-07"
+                 iyy="2.234728e-05" iyz="0.000000e+00"
+                 izz="1.965878e-05" />
       </inertial>
     </link>
@@ -51,5 +48,5 @@
       <origin xyz="0.012 0.0 0.017" rpy="0 0 0"/>
       <axis xyz="0 0 1"/>
-      <limit velocity="4.8" effort="1.5" lower="${-pi}" upper="${pi}" />
+      <limit velocity="4.8" effort="1.5" lower="${-3*pi/4}" upper="${3*pi/4}" />
       <dynamics damping="0.1"/>
     </joint>
@@ -68,12 +65,11 @@
         </geometry>
       </collision>
-      <!-- link2 — Joint 1 del PDF (masa ensamble motor+eslabon).
-           R = I (C1 frame alineado con URDF link2 frame). -->
-      <inertial>
-        <origin xyz="0.0000000e+00 -5.6914372e-04 2.6565513e-02" rpy="0 0 0"/>
-        <mass value="1.0483260e-01" />
-        <inertia ixx="3.3802078e-05" ixy="0.0"           ixz="0.0"
-                 iyy="2.9569411e-05" iyz="2.2121514e-07"
-                 izz="1.7810252e-05" />
+      <!-- link2 — balanza + Inventor CAD (escalado m_real/m_CAD) -->
+      <inertial>
+        <origin xyz="0.000000 0.000657 0.044319" rpy="0 0 0"/>
+        <mass value="0.0970" />
+        <inertia ixx="3.078317e-05" ixy="0.000000e+00" ixz="0.000000e+00"
+                 iyy="2.670366e-05" iyz="-1.289659e-07"
+                 izz="1.627175e-05" />
       </inertial>
     </link>
@@ -83,5 +79,5 @@
       <origin xyz="0.0 0.0 0.0595" rpy="0 0 0"/>
       <axis xyz="0 1 0"/>
-      <limit velocity="4.8" effort="1.5" lower="${-1.5}" upper="${1.5}" />
+      <limit velocity="4.8" effort="1.5" lower="${-11*pi/18}" upper="${5*pi/9}" />
       <dynamics damping="0.1"/>
     </joint>
@@ -100,12 +96,11 @@
         </geometry>
       </collision>
-      <!-- link3 — Joint 2 del PDF.
-           R = Rz(180 deg): r_urdf = (-x_C, -y_C, z_C); Ixz->-Ixz, Iyz->-Iyz. -->
-      <inertial>
-        <origin xyz="9.1617228e-03 4.1915210e-04 1.0599938e-01" rpy="0 0 0"/>
-        <mass value="1.4234630e-01" />
-        <inertia ixx="2.3711450e-04" ixy="-2.7513999e-07" ixz="-2.6668982e-05"
-                 iyy="2.4488355e-04" iyz="-1.3128636e-06"
-                 izz="4.2967059e-05" />
+      <!-- link3 — balanza + Inventor CAD (escalado m_real/m_CAD) -->
+      <inertial>
+        <origin xyz="0.007606 0.000389 0.099924" rpy="0 0 0"/>
+        <mass value="0.1235" />
+        <inertia ixx="1.979680e-04" ixy="-2.511443e-07" ixz="-2.497601e-05"
+                 iyy="2.046627e-04" iyz="-1.351040e-06"
+                 izz="3.374865e-05" />
       </inertial>
     </link>
@@ -115,5 +110,5 @@
       <origin xyz="0.024 0 0.128" rpy="0 0 0"/>
       <axis xyz="0 1 0"/>
-      <limit velocity="4.8" effort="1.5" lower="${-1.5}" upper="${1.4}" />
+      <limit velocity="4.8" effort="1.5" lower="${-11*pi/18}" upper="${pi/2}" />
       <dynamics damping="0.1"/>
     </joint>
@@ -132,13 +127,11 @@
         </geometry>
       </collision>
-      <!-- link4 — Joint 3 del PDF.
-           R = R_alt: C3_z->URDF_x, C3_y->-URDF_y, C3_x->+URDF_z.
-           I_urdf = [Izz,-Iyz,Ixz; -Iyz,Iyy,-Ixy; Ixz,-Ixy,Ixx]. -->
-      <inertial>
-        <origin xyz="9.3290225e-02 4.4304274e-04 3.6312773e-07" rpy="0 0 0"/>
-        <mass value="1.3467049e-01" />
-        <inertia ixx="2.4809204e-05" ixy="-1.2221090e-06" ixz="1.8290300e-09"
-                 iyy="1.7818139e-04" iyz="0.0"
-                 izz="1.8688812e-04" />
+      <!-- link4 — balanza + Inventor CAD (escalado m_real/m_CAD) -->
+      <inertial>
+        <origin xyz="0.089168 0.000437 0.000001" rpy="0 0 0"/>
+        <mass value="0.1151" />
+        <inertia ixx="1.930305e-05" ixy="-1.189078e-06" ixz="3.461654e-09"
+                 iyy="1.483284e-04" iyz="0.000000e+00"
+                 izz="1.547550e-04" />
       </inertial>
     </link>
@@ -148,5 +141,5 @@
       <origin xyz="0.124 0.0 0.0" rpy="0 0 0"/>
       <axis xyz="0 1 0"/>
-      <limit velocity="4.8" effort="1.5" lower="${-1.7}" upper="${1.97}" />
+      <limit velocity="4.8" effort="1.5" lower="-1.8" upper="2.1" />
       <dynamics damping="0.1"/>
     </joint>
@@ -165,13 +158,11 @@
         </geometry>
       </collision>
-      <!-- link5 — Joint 4 del PDF (incluye motor + ensamble de muneca/gripper).
-           R = R_alt: C4_z->URDF_x, C4_y->-URDF_y, C4_x->+URDF_z.
-           I_urdf = [Izz,-Iyz,Ixz; -Iyz,Iyy,-Ixy; Ixz,-Ixy,Ixx]. -->
-      <inertial>
-        <origin xyz="6.0472935e-02 7.9503949e-07 6.1273313e-03" rpy="0 0 0"/>
-        <mass value="2.3650927e-01" />
-        <inertia ixx="1.7393236e-04" ixy="-1.5305492e-08" ixz="2.2615865e-05"
-                 iyy="2.0769766e-04" iyz="-2.2288943e-07"
-                 izz="2.6708326e-04" />
+      <!-- link5 — balanza + Inventor CAD (escalado m_real/m_CAD) -->
+      <inertial>
+        <origin xyz="0.062451 0.000000 0.005878" rpy="0 0 0"/>
+        <mass value="0.2206" />
+        <inertia ixx="1.344328e-04" ixy="-1.788649e-08" ixz="2.259163e-05"
+                 iyy="1.892619e-04" iyz="9.936937e-07"
+                 izz="2.174510e-04" />
       </inertial>
     </link>

Commit message: Mallas del robot: usar meshes/ propio en vez de open_manipulator_x_description
El URDF y el xacro apuntaban a paquetes externos (open_manipulator_description
sin _x con nombres chain_link*.stl, y open_manipulator_x_description) para
resolver las mallas de los links. Ahora usan las mallas locales del paquete
(meshes/link1..5.stl, gripper_left_palm.stl, gripper_right_palm.stl).

Se agrega la exportacion gazebo_ros gazebo_model_path en package.xml, requerida
por ros_gz_sim/gz_sim.launch.py para incluir este paquete en GZ_SIM_RESOURCE_PATH;
sin ella Gazebo Fortress no resuelve las URIs model://open_manipulator_x_torque_control/...
y las mallas no se renderizan en la simulacion.

Co-Authored-By: Claude Sonnet 5 <noreply@anthropic.com>

File: urdf/open_manipulator_x.urdf (robot description, URDF)
Before this commit: robot open_manipulator, 8 links, 7 joints
Links:
- link gripper_link: geometry collision mesh filename=package://open_manipulator_x_torque_control/meshes/gripper_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 scale=0.001 0.001 0.001; visual mesh filename=package://open_manipulator_x_torque_control/meshes/gripper_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 scale=0.001 0.001 0.001
- link gripper_link_sub: geometry collision mesh filename=package://open_manipulator_x_torque_control/meshes/gripper_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 scale=0.001 0.001 0.001; visual mesh filename=package://open_manipulator_x_torque_control/meshes/gripper_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 scale=0.001 0.001 0.001
- link link1: geometry collision mesh filename=package://open_manipulator_x_torque_control/meshes/link1.stl scale=0.001 0.001 0.001; visual mesh filename=package://open_manipulator_x_torque_control/meshes/link1.stl scale=0.001 0.001 0.001
- link link2: geometry collision mesh filename=package://open_manipulator_x_torque_control/meshes/link2.stl scale=0.001 0.001 0.001; visual mesh filename=package://open_manipulator_x_torque_control/meshes/link2.stl scale=0.001 0.001 0.001
- link link3: geometry collision mesh filename=package://open_manipulator_x_torque_control/meshes/link3.stl scale=0.001 0.001 0.001; visual mesh filename=package://open_manipulator_x_torque_control/meshes/link3.stl scale=0.001 0.001 0.001
- link link4: geometry collision mesh filename=package://open_manipulator_x_torque_control/meshes/link4.stl scale=0.001 0.001 0.001; visual mesh filename=package://open_manipulator_x_torque_control/meshes/link4.stl scale=0.001 0.001 0.001
- link link5: geometry collision mesh filename=package://open_manipulator_x_torque_control/meshes/link5.stl scale=0.001 0.001 0.001; visual mesh filename=package://open_manipulator_x_torque_control/meshes/link5.stl scale=0.001 0.001 0.001

File: xacro/open_manipulator_x.urdf.xacro (robot description, xacro)
@@ -13,6 +13,7 @@
     damping_scale      : factor multiplicativo para damping de joint1..joint4
     friction_scale     : factor multiplicativo para friction de joint1..joint4
+  Cambios adicionales:
+    - Meshes: ahora se cargan desde este mismo paquete (meshes/), ya no desde open_manipulator_x_description
   Sin cambios:
-    - Meshes (mismo paquete open_manipulator_x_description)
     - Origenes y ejes articulares
     - Gripper links inertial (masa dummy)
@@ -24,5 +25,5 @@
     <xacro:property
       name="meshes_file_direction"
-      value="package://open_manipulator_x_description/meshes"/>
+      value="package://open_manipulator_x_torque_control/meshes"/>
     <link name="${prefix}link1">
       <visual>
